Commit message: In order to visualize the urdf model in vrep, change the joint and link names of urdf model to make it consistency with vrep model.

File: include/grl/flatbuffer/Robone_KukaLBRiiwa.urdf (robot description, URDF)
Before this commit: robot iiwa14, 11 links, 10 joints
Links:
- removed link iiwa_link_0
- removed link iiwa_link_1
- removed link iiwa_link_2
- removed link iiwa_link_3
- removed link iiwa_link_4
- removed link iiwa_link_5
- removed link iiwa_link_6
- removed link iiwa_link_7
- removed link iiwa_link_ee
- removed link iiwa_link_marker
- added link LBR_iiwa_14_R820_link0, mass 5; collision mesh filename=package://iiwa_description/meshes/iiwa14/collision/link_0.s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; visual mesh filename=package://iiwa_description/meshes/iiwa14/visual/link_0.stl
- added link LBR_iiwa_14_R820_link1, mass 4; collision mesh filename=package://iiwa_description/meshes/iiwa14/collision/link_1.s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; visual mesh filename=package://iiwa_description/meshes/iiwa14/visual/link_1.stl
- added link LBR_iiwa_14_R820_link2, mass 4; collision mesh filename=package://iiwa_description/meshes/iiwa14/collision/link_2.s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; visual mesh filename=package://iiwa_description/meshes/iiwa14/visual/link_2.stl
- added link LBR_iiwa_14_R820_link3, mass 3; collision mesh filename=package://iiwa_description/meshes/iiwa14/collision/link_3.s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; visual mesh filename=package://iiwa_description/meshes/iiwa14/visual/link_3.stl
- added link LBR_iiwa_14_R820_link4, mass 2.7; collision mesh filename=package://iiwa_description/meshes/iiwa14/collision/link_4.s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; visual mesh filename=package://iiwa_description/meshes/iiwa14/visual/link_4.stl
- added link LBR_iiwa_14_R820_link5, mass 1.7; collision mesh filename=package://iiwa_description/meshes/iiwa14/collision/link_5.s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; visual mesh filename=package://iiwa_description/meshes/iiwa14/visual/link_5.stl
- added link LBR_iiwa_14_R820_link6, mass 1.8; collision mesh filename=package://iiwa_description/meshes/iiwa14/collision/link_6.s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; visual mesh filename=package://iiwa_description/meshes/iiwa14/visual/link_6.stl
- added link LBR_iiwa_14_R820_link7, mass 0.3; collision mesh filename=package://iiwa_description/meshes/iiwa14/collision/link_7.s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; visual mesh filename=package://iiwa_description/meshes/iiwa14/visual/link_7.stl
- added link LBR_iiwa_14_R820_link_marker
- added link RobotFlangeTip
Joints:
- removed joint iiwa_joint_1
- removed joint iiwa_joint_2
- removed joint iiwa_joint_3
- removed joint iiwa_joint_4
- removed joint iiwa_joint_5
- removed joint iiwa_joint_6
- removed joint iiwa_joint_7
- removed joint iiwa_joint_ee
- removed joint iiwa_joint_marker
- removed joint world_iiwa_joint
- added joint LBR_iiwa_14_R820_joint1: type revolute, parent LBR_iiwa_14_R820_link0, child LBR_iiwa_14_R820_link1, origin xyz=0 0 0.1575 rpy=0 0 0, axis 0 0 1, limit lower=-2.96705972839 upper=2.96705972839 effort=300 velocity=10
- added joint LBR_iiwa_14_R820_joint2: type revolute, parent LBR_iiwa_14_R820_link1, child LBR_iiwa_14_R820_link2, origin xyz=0 0 0.2025 rpy=1.57079632679   0 3.14159265359, axis 0 0 1, limit lower=-2.09439510239 upper=2.09439510239 effort=300 velocity=10
- added joint LBR_iiwa_14_R820_joint3: type revolute, parent LBR_iiwa_14_R820_link2, child LBR_iiwa_14_R820_link3, origin xyz=0 0.2045 0 rpy=1.57079632679 0 3.14159265359, axis 0 0 1, limit lower=-2.96705972839 upper=2.96705972839 effort=300 velocity=10
- added joint LBR_iiwa_14_R820_joint4: type revolute, parent LBR_iiwa_14_R820_link3, child LBR_iiwa_14_R820_link4, origin xyz=0 0 0.2155 rpy=1.57079632679 0 0, axis 0 0 1, limit lower=-2.09439510239 upper=2.09439510239 effort=300 velocity=10
- added joint LBR_iiwa_14_R820_joint5: type revolute, parent LBR_iiwa_14_R820_link4, child LBR_iiwa_14_R820_link5, origin xyz=0 0.1845 0 rpy=-1.57079632679 3.14159265359 0, axis 0 0 1, limit lower=-2.96705972839 upper=2.96705972839 effort=300 velocity=10
- added joint LBR_iiwa_14_R820_joint6: type revolute, parent LBR_iiwa_14_R820_link5, child LBR_iiwa_14_R820_link6, origin xyz=0 0 0.2155 rpy=1.57079632679 0 0, axis 0 0 1, limit lower=-2.09439510239 upper=2.09439510239 effort=300 velocity=10
- added joint LBR_iiwa_14_R820_joint7: type revolute, parent LBR_iiwa_14_R820_link6, child LBR_iiwa_14_R820_link7, origin xyz=0 0.081 0 rpy=-1.57079632679 3.14159265359 0, axis 0 0 1, limit lower=-3.05432619099 upper=3.05432619099 effort=300 velocity=10
- added joint LBR_iiwa_14_R820_joint_ee: type fixed, parent LBR_iiwa_14_R820_link7, child RobotFlangeTip, origin xyz=0 0 0.045 rpy=0 0 0
- added joint LBR_iiwa_14_R820_joint_marker: type fixed, parent RobotFlangeTip, child LBR_iiwa_14_R820_link_marker, origin xyz=0.052998 0.090310 0.090627 rpy=0 0 0
- added joint world_LBR_iiwa_14_R820_joint: type fixed, parent world, child LBR_iiwa_14_R820_link0, origin xyz=0 0 0 rpy=0 0 0
